Commit message: Update mass and effort values in URDF for kuka_kr300r2500ultra model

File: urdf/kr300r2500ultra_macro.xacro (robot description, xacro)
@@ -8,5 +8,5 @@
       <inertial>
         <origin xyz="0 0 0" rpy="0 0 0"/>
-        <mass value="2"/>
+        <mass value="2.2596E2"/>
         <inertia ixx="0.01" ixy="0" ixz="0" iyy="0.01" iyz="0" izz="0.01" />
       </inertial>
@@ -31,5 +31,5 @@
       <inertial>
         <origin xyz="0 0 0" rpy="0 0 0"/>
-        <mass value="2"/>
+        <mass value="3.6737E2"/>
         <inertia ixx="0.01" ixy="0" ixz="0" iyy="0.01" iyz="0" izz="0.01" />
       </inertial>
@@ -54,5 +54,5 @@
       <inertial>
         <origin xyz="0 0 0" rpy="0 0 0"/>
-        <mass value="2"/>
+        <mass value="2.3206E2"/>
         <inertia ixx="0.01" ixy="0" ixz="0" iyy="0.01" iyz="0" izz="0.01" />
       </inertial>
@@ -77,5 +77,5 @@
       <inertial>
         <origin xyz="0 0 0" rpy="0 0 0"/>
-        <mass value="2"/>
+        <mass value="1.9153E2"/>
         <inertia ixx="0.01" ixy="0" ixz="0" iyy="0.01" iyz="0" izz="0.01" />
       </inertial>
@@ -100,5 +100,5 @@
       <inertial>
         <origin xyz="0 0 0" rpy="0 0 0"/>
-        <mass value="2"/>
+        <mass value="4.7942845677E1"/>
         <inertia ixx="0.01" ixy="0" ixz="0" iyy="0.01" iyz="0" izz="0.01" />
       </inertial>
@@ -123,5 +123,5 @@
       <inertial>
         <origin xyz="0 0 0" rpy="0 0 0"/>
-        <mass value="2"/>
+        <mass value="2.3687644624E1"/>
         <inertia ixx="0.01" ixy="0" ixz="0" iyy="0.01" iyz="0" izz="0.01" />
       </inertial>
@@ -146,5 +146,5 @@
       <inertial>
         <origin xyz="0 0 0" rpy="0 0 0"/>
-        <mass value="2"/>
+        <mass value="1.2245718539E1"/>
         <inertia ixx="0.01" ixy="0" ixz="0" iyy="0.01" iyz="0" izz="0.01" />
       </inertial>
@@ -176,5 +176,5 @@
       <child link="${prefix}link_1"/>
       <axis xyz="0 0 -1"/>
-      <limit effort="0" lower="${-DEG2RAD * 185}" upper="${DEG2RAD * 185}" velocity="${DEG2RAD * 156}"/>
+      <limit effort="7.29E3" lower="${-DEG2RAD * 185}" upper="${DEG2RAD * 185}" velocity="${DEG2RAD * 156}"/>
     </joint>
     <!-- joint 2 (A2) -->
@@ -184,5 +184,5 @@
       <child link="${prefix}link_2"/>
       <axis xyz="0 1 0"/>
-      <limit effort="0" lower="${-DEG2RAD * 155}" upper="${DEG2RAD * 35}" velocity="${DEG2RAD * 156}"/>
+      <limit effort="9.60003E3" lower="${-DEG2RAD * 155}" upper="${DEG2RAD * 35}" velocity="${DEG2RAD * 156}"/>
     </joint>
     <!-- joint 3 (A3) -->
@@ -192,5 +192,5 @@
       <child link="${prefix}link_3"/>
       <axis xyz="0 1 0"/>
-      <limit effort="0" lower="${-DEG2RAD * 130}" upper="${DEG2RAD * 154}" velocity="${DEG2RAD * 156}"/>
+      <limit effort="7.08714342281144E3" lower="${-DEG2RAD * 130}" upper="${DEG2RAD * 154}" velocity="${DEG2RAD * 156}"/>
     </joint>
     <!-- joint 4 (A4) -->
@@ -200,5 +200,5 @@
       <child link="${prefix}link_4"/>
       <axis xyz="-1 0 0"/>
-      <limit effort="0" lower="${-DEG2RAD * 350}" upper="${DEG2RAD * 350}" velocity="${DEG2RAD * 330}"/>
+      <limit effort="2.25887888718356E3" lower="${-DEG2RAD * 350}" upper="${DEG2RAD * 350}" velocity="${DEG2RAD * 330}"/>
     </joint>
     <!-- joint 5 (A5) -->
@@ -208,5 +208,5 @@
       <child link="${prefix}link_5"/>
       <axis xyz="0 1 0"/>
-      <limit effort="0" lower="${-DEG2RAD * 130}" upper="${DEG2RAD * 130}" velocity="${DEG2RAD * 330}"/>
+      <limit effort="2.26120660090655E3" lower="${-DEG2RAD * 130}" upper="${DEG2RAD * 130}" velocity="${DEG2RAD * 330}"/>
     </joint>
     <!-- joint 6 (A6) -->
@@ -216,5 +216,5 @@
       <child link="${prefix}link_6"/>
       <axis xyz="-1 0 0"/>
-      <limit effort="0" lower="${-DEG2RAD * 350}" upper="${DEG2RAD * 350}" velocity="${DEG2RAD * 615}"/>
+      <limit effort="1.46107811041986E3" lower="${-DEG2RAD * 350}" upper="${DEG2RAD * 350}" velocity="${DEG2RAD * 615}"/>
     </joint>
     <!-- tool frame - fixed frame -->

Commit message: fix(urdf): add flange following ROS REP-103 and redefine tool0 for controller alignment

File: urdf/kr300r2500ultra_macro.xacro (robot description, xacro)
@@ -165,4 +165,6 @@
       </collision>
     </link>
+    <!-- flange -->
+    <link name="${prefix}flange"/>
     <!-- tool 0 -->
     <!-- This frame corresponds to the $FLANGE coordinate system in KUKA KRC controllers. -->
@@ -218,9 +220,15 @@
       <limit effort="1.46107811041986E3" lower="${-DEG2RAD * 350}" upper="${DEG2RAD * 350}" velocity="${DEG2RAD * 615}"/>
     </joint>
+    <!-- flange -->
+    <joint name="${prefix}joint_a6-flange" type="fixed">
+      <parent link="${prefix}link_6"/>
+      <child link="${prefix}flange"/>
+      <origin xyz="0.240 0 0" rpy="0 0 0"/>
+    </joint>
     <!-- tool frame - fixed frame -->
-    <joint name="${prefix}joint_a6-tool0" type="fixed">
-      <parent link="${prefix}link_6"/>
+    <joint name="${prefix}flange-tool0" type="fixed">
+      <parent link="${prefix}flange"/>
       <child link="${prefix}tool0"/>
-      <origin xyz="0.240 0 0" rpy="0 ${DEG2RAD * 90} 0"/>
+      <origin xyz="0 0 0" rpy="0 ${DEG2RAD * 90} 0"/>
     </joint>
     <!-- END JOINTS -->
